Commit message: Enhance motion planning capabilities with new nodes and parameters
- Added new nodes for MoveIt Cartesian planning and test planner pose in setup.py.
- Updated exclusion zone configurations in ur3e_workspace.yaml for improved collision detection.
- Refactored motion planning launch file to support multiple planning backends: RMRC, MoveIt OMPL, and MoveIt Cartesian.
- Introduced new launch parameters for MoveIt Cartesian planning, including max_step, jump_threshold, and collision avoidance settings.
- Enhanced PoseGoalNode to publish status updates and track execution phases.
- Updated RMRC planning node parameters for better control over execution and kinematics.

File: src/ur3e_controller/urdf/ur3e_workspace.urdf.xacro (robot description, xacro)
@@ -106,5 +106,5 @@
     trajectory_port="$(arg trajectory_port)"
     >
-    <origin xyz="0 0 $(arg base_height)" rpy="0 0 0"/>
+    <origin xyz="0 0 $(arg base_height)" rpy="0 0 ${-pi/2}"/>
   </xacro:ur_robot>
   <xacro:if value="$(arg sim_gazebo)">
